Commit message: injerrobot_description: removed ur arms

File: injerrobot_description/robots/injerrobot_platform.urdf.xacro (robot description, xacro)
@@ -8,9 +8,6 @@
   <!-- Import Kuka KR6900 -->
   <xacro:include filename="$(find kuka_kr6_support)/urdf/kr6r900sixx_macro.xacro" />
-  <!-- Import UR10 -->
-  <xacro:include filename="$(find ur_description)/urdf/ur10.urdf.xacro"/>
   <!-- Import common gazebo elements -->
   <xacro:include filename="$(find injerrobot_description)/robots/common.gazebo.xacro" />
-  <xacro:property name="load_ur" value="false" />
   <link name="world" />
   <!-- Fix left arm to world link -->
@@ -26,12 +23,6 @@
     <child link="right_arm_base_link"/>
   </joint>
-  <xacro:unless value="${load_ur}">
-    <xacro:kuka_kr6r900sixx prefix="right_arm_"/>
-    <xacro:kuka_kr6r900sixx prefix="left_arm_"/>
-  </xacro:unless>
-  <xacro:if value="${load_ur}">
-    <xacro:ur10_robot prefix="right_arm_" joint_limited="true"/>
-    <xacro:ur10_robot prefix="left_arm_" joint_limited="true"/>
-  </xacro:if>
+  <xacro:kuka_kr6r900sixx prefix="right_arm_"/>
+  <xacro:kuka_kr6r900sixx prefix="left_arm_"/>
   <xacro:ros_control />
 </robot>

Commit message: injerrobot_description: added cell models

File: injerrobot_description/robots/injerrobot_platform.urdf.xacro (robot description, xacro)
@@ -8,21 +8,109 @@
   <!-- Import Kuka KR6900 -->
   <xacro:include filename="$(find kuka_kr6_support)/urdf/kr6r900sixx_macro.xacro" />
+  <xacro:include filename="$(find injerrobot_description)/urdf/conveyor.urdf.xacro" />
+  <xacro:include filename="$(find injerrobot_description)/urdf/gripper.urdf.xacro" />
+  <xacro:include filename="$(find injerrobot_description)/urdf/clipper.urdf.xacro" />
   <!-- Import common gazebo elements -->
   <xacro:include filename="$(find injerrobot_description)/robots/common.gazebo.xacro" />
   <link name="world" />
   <!-- Fix left arm to world link -->
-  <joint name="left_arm_base_joint" type="fixed">
-    <origin xyz="0 0.5 0" rpy="0 0 0 "/>  <!-- TODO: set correct orientation -->
+  <joint name="left_arm_floor_joint" type="fixed"> <!-- R1, rootstock -->
+    <origin xyz="0 0 0" rpy="0 0 0 "/>
     <parent link="world"/>
+    <child link="left_arm_floor_link"/>
+  </joint>
+  <link name="left_arm_floor_link">
+    <visual>
+        <origin xyz="0 0 0.5" rpy="0 0 0"/>
+        <geometry>
+            <box size="0.4 0.3 1.0" />
+        </geometry>
+        <material name="grey">
+            <color rgba="0.5 0.5 0.5 1.0"/>
+        </material>
+  </visual>
+  <collision>
+    <origin xyz="0 0 0.5" rpy="0 0 0"/>
+        <geometry>
+            <box size="0.4 0.3 1.0" />
+        </geometry>
+        <material name="red">
+            <color rgba="1.0 0.0 0.0 1.0"/>
+        </material>
+    </collision>
+  </link>
+  <joint name="left_arm_base_joint" type="fixed"> <!-- R1, rootstock -->
+    <origin xyz="0 0 1.0" rpy="0 0 0 "/>
+    <parent link="left_arm_floor_link"/>
     <child link="left_arm_base_link"/>
   </joint>
   <!-- Fix right arm to world link -->
-  <joint name="right_arm_base_joint" type="fixed">
-    <origin xyz="0 -0.5 0" rpy="0 0 0 "/>  <!-- TODO: set correct orientation -->
+  <joint name="right_arm_floor_joint" type="fixed"> <!-- R2, scion -->
+    <origin xyz="1.9 0 0.0" rpy="0 0 -${PI/2.0}"/>
     <parent link="world"/>
+    <child link="right_arm_floor_link"/>
+  </joint>
+  <link name="right_arm_floor_link">
+    <visual>
+        <origin xyz="0 0 0.5" rpy="0 0 0"/>
+        <geometry>
+            <box size="0.4 0.3 1.0" />
+        </geometry>
+        <material name="grey">
+            <color rgba="0.5 0.5 0.5 1.0"/>
+        </material>
+  </visual>
+  <collision>
+    <origin xyz="0 0 0.5" rpy="0 0 0"/>
+        <geometry>
+            <box size="0.4 0.3 1.0" />
+        </geometry>
+        <material name="red">
+            <color rgba="1.0 0.0 0.0 1.0"/>
+        </material>
+    </collision>
+  </link>
+  <joint name="right_arm_base_joint" type="fixed"> <!-- R1, rootstock -->
+    <origin xyz="0 0 1.0" rpy="0 0 0 "/>
+    <parent link="right_arm_floor_link"/>
     <child link="right_arm_base_link"/>
   </joint>
+  <!-- Fix left arm to world link -->
+  <joint name="clipper_floor_joint" type="fixed"> <!-- R1, rootstock -->
+    <origin xyz="1.0 0.5 0" rpy="0 0 1.5707 "/>
+    <parent link="world"/>
+    <child link="clipper_floor_link"/>
+  </joint>
+  <link name="clipper_floor_link">
+    <visual>
+        <origin xyz="0 0 0.5" rpy="0 0 0"/>
+        <geometry>
+            <box size="0.4 0.3 1.0" />
+        </geometry>
+        <material name="grey">
+            <color rgba="0.5 0.5 0.5 1.0"/>
+        </material>
+  </visual>
+  </link>
+    <joint name="clipper_base_joint" type="fixed"> <!-- R1, rootstock -->
+    <origin xyz="0 0 1.0" rpy="0 0 0 "/>
+    <parent link="clipper_floor_link"/>
+    <child link="clipper_base_link"/>
+  </joint>
+  <link name="clipper_base_link" />
+  <xacro:clipper prefix="" parent="clipper_base_link"/>
   <xacro:kuka_kr6r900sixx prefix="right_arm_"/>
+  <xacro:gripper prefix="right_arm_" parent="right_arm_link_6" />
   <xacro:kuka_kr6r900sixx prefix="left_arm_"/>
+  <xacro:gripper prefix="left_arm_" parent="left_arm_link_6" />
+  <xacro:conveyor prefix="rootstock_feeder_" parent="left_arm_floor_link">
+        <origin xyz="-0.318 0.800 0" rpy="0 0 0"/>
+  </xacro:conveyor>
+  <xacro:conveyor prefix="rootstock_dispenser_" parent="left_arm_floor_link">
+        <origin xyz="-0.318 -0.800 0" rpy="0 0 0"/>
+  </xacro:conveyor>
+  <xacro:conveyor prefix="scion_feeder_" parent="right_arm_floor_link">
+        <origin xyz="0.239 0.712 0" rpy="0 0 0"/>
+  </xacro:conveyor>
   <xacro:ros_control />
 </robot>

Commit message: injerrobot_description: updated platform model and added plinth

File: injerrobot_description/robots/injerrobot_platform.urdf.xacro (robot description, xacro)
@@ -11,104 +11,41 @@
   <xacro:include filename="$(find injerrobot_description)/urdf/gripper.urdf.xacro" />
   <xacro:include filename="$(find injerrobot_description)/urdf/clipper.urdf.xacro" />
+  <xacro:include filename="$(find injerrobot_description)/urdf/plinth.urdf.xacro" />
   <!-- Import common gazebo elements -->
   <xacro:include filename="$(find injerrobot_description)/robots/common.gazebo.xacro" />
   <link name="world" />
   <!-- Fix left arm to world link -->
-  <joint name="left_arm_floor_joint" type="fixed"> <!-- R1, rootstock -->
-    <origin xyz="0 0 0" rpy="0 0 0 "/>
-    <parent link="world"/>
-    <child link="left_arm_floor_link"/>
-  </joint>
-  <link name="left_arm_floor_link">
-    <visual>
-        <origin xyz="0 0 0.5" rpy="0 0 0"/>
-        <geometry>
-            <box size="0.4 0.3 1.0" />
-        </geometry>
-        <material name="grey">
-            <color rgba="0.5 0.5 0.5 1.0"/>
-        </material>
-  </visual>
-  <collision>
-    <origin xyz="0 0 0.5" rpy="0 0 0"/>
-        <geometry>
-            <box size="0.4 0.3 1.0" />
-        </geometry>
-        <material name="red">
-            <color rgba="1.0 0.0 0.0 1.0"/>
-        </material>
-    </collision>
-  </link>
+  <xacro:plinth prefix="left_arm_" height="1.0" parent="world">
+      <origin xyz="0 0 0" rpy="0 0 0"/>
+  </xacro:plinth>
+  <xacro:plinth prefix="right_arm_" height="1.0" parent="world">
+      <origin xyz="1.3 0 0.0" rpy="0 0 -${PI/2.0}"/>
+  </xacro:plinth>
+  <xacro:plinth prefix="clipper_" height="1.0" parent="world">
+    <origin xyz="1.0 0.5 0" rpy="0 0 -1.57 "/>
+  </xacro:plinth>
+  <!-- Fix left arm to world link -->
+  <xacro:clipper prefix="" parent="clipper_plinth_link"/>
   <joint name="left_arm_base_joint" type="fixed"> <!-- R1, rootstock -->
-    <origin xyz="0 0 1.0" rpy="0 0 0 "/>
-    <parent link="left_arm_floor_link"/>
+    <origin xyz="0 0 0.0" rpy="0 0 0 "/>
+    <parent link="left_arm_plinth_link"/>
     <child link="left_arm_base_link"/>
   </joint>
-  <!-- Fix right arm to world link -->
-  <joint name="right_arm_floor_joint" type="fixed"> <!-- R2, scion -->
-    <origin xyz="1.9 0 0.0" rpy="0 0 -${PI/2.0}"/>
-    <parent link="world"/>
-    <child link="right_arm_floor_link"/>
-  </joint>
-  <link name="right_arm_floor_link">
-    <visual>
-        <origin xyz="0 0 0.5" rpy="0 0 0"/>
-        <geometry>
-            <box size="0.4 0.3 1.0" />
-        </geometry>
-        <material name="grey">
-            <color rgba="0.5 0.5 0.5 1.0"/>
-        </material>
-  </visual>
-  <collision>
-    <origin xyz="0 0 0.5" rpy="0 0 0"/>
-        <geometry>
-            <box size="0.4 0.3 1.0" />
-        </geometry>
-        <material name="red">
-            <color rgba="1.0 0.0 0.0 1.0"/>
-        </material>
-    </collision>
-  </link>
-  <joint name="right_arm_base_joint" type="fixed"> <!-- R1, rootstock -->
-    <origin xyz="0 0 1.0" rpy="0 0 0 "/>
-    <parent link="right_arm_floor_link"/>
+  <joint name="right_arm_base_joint" type="fixed"> <!-- R2, scion -->
+    <origin xyz="0 0 0.0" rpy="0 0 0 "/>
+    <parent link="right_arm_plinth_link"/>
     <child link="right_arm_base_link"/>
   </joint>
-  <!-- Fix left arm to world link -->
-  <joint name="clipper_floor_joint" type="fixed"> <!-- R1, rootstock -->
-    <origin xyz="1.0 0.5 0" rpy="0 0 1.5707 "/>
-    <parent link="world"/>
-    <child link="clipper_floor_link"/>
-  </joint>
-  <link name="clipper_floor_link">
-    <visual>
-        <origin xyz="0 0 0.5" rpy="0 0 0"/>
-        <geometry>
-            <box size="0.4 0.3 1.0" />
-        </geometry>
-        <material name="grey">
-            <color rgba="0.5 0.5 0.5 1.0"/>
-        </material>
-  </visual>
-  </link>
-    <joint name="clipper_base_joint" type="fixed"> <!-- R1, rootstock -->
-    <origin xyz="0 0 1.0" rpy="0 0 0 "/>
-    <parent link="clipper_floor_link"/>
-    <child link="clipper_base_link"/>
-  </joint>
-  <link name="clipper_base_link" />
-  <xacro:clipper prefix="" parent="clipper_base_link"/>
   <xacro:kuka_kr6r900sixx prefix="right_arm_"/>
-  <xacro:gripper prefix="right_arm_" parent="right_arm_link_6" />
+  <!-- xacro:gripper prefix="right_arm_" parent="right_arm_link_6" /-->
   <xacro:kuka_kr6r900sixx prefix="left_arm_"/>
-  <xacro:gripper prefix="left_arm_" parent="left_arm_link_6" />
-  <xacro:conveyor prefix="rootstock_feeder_" parent="left_arm_floor_link">
+  <!-- xacro:gripper prefix="left_arm_" parent="left_arm_link_6" /-->
+  <xacro:conveyor prefix="rootstock_feeder_" parent="left_arm_plinth_base_link">
         <origin xyz="-0.318 0.800 0" rpy="0 0 0"/>
   </xacro:conveyor>
-  <xacro:conveyor prefix="rootstock_dispenser_" parent="left_arm_floor_link">
+  <xacro:conveyor prefix="rootstock_dispenser_" parent="left_arm_plinth_base_link">
         <origin xyz="-0.318 -0.800 0" rpy="0 0 0"/>
   </xacro:conveyor>
-  <xacro:conveyor prefix="scion_feeder_" parent="right_arm_floor_link">
+  <xacro:conveyor prefix="scion_feeder_" parent="right_arm_plinth_base_link">
         <origin xyz="0.239 0.712 0" rpy="0 0 0"/>
   </xacro:conveyor>
